File: tsal-ups.kicad_sch (KiCad schematic)
At the start: 56 parts, among them J3 UPS Battery Connector, J4 +12V, J5 +12V_OUT, Q3 2N7002, Q4 2N7002, Q5 2N7002, Q6 2N7002, Q7 2N7002, U1 TPS552892RYQR, U2 TPS2121RUXR

Commit message: Revision A
Parts:
- removed C7: 10u, symbol Device:C
- removed C9: 50u, symbol Device:C_Polarized
- removed R19, R20: R, symbol Device:R
- removed TP1, TP4: TestPoint_2Pole, yfs:TestPoint_2Pads_Pitch2.54mm_Drill1.0mm, symbol Connector:TestPoint_2Pole
- added C10: 22u, Capacitor_SMD:CP_Elec_6.3x7.7, symbol Device:C_Polarized
- added C16, C19: 1u, Capacitor_SMD:C_0603_1608Metric, symbol Device:C
- added C17: 100u, Capacitor_SMD:CP_Elec_6.3x7.7, symbol Device:C_Polarized
- added C9: 4.7u, Capacitor_SMD:C_0805_2012Metric, symbol Device:C
- added D2, D6: BZX384C20, Diode_SMD:D_SOD-323, symbol Diode:BZX384xxxx
- added H1, H2, H3, H4: MountingHole_Pad, MountingHole:MountingHole_3.2mm_M3_Pad_Via, symbol Mechanical:MountingHole_Pad
- added R18: 24k, Resistor_SMD:R_0603_1608Metric, symbol Device:R
- added R21: 3.3k, Resistor_SMD:R_0603_1608Metric, symbol Device:R
- added TP10, TP11, TP3, TP4, TP5, TP6, TP7, TP8, TP9: TestPoint, TestPoint:TestPoint_Pad_D1.5mm, symbol Connector:TestPoint
- C1: footprint (none) -> Capacitor_SMD:C_0603_1608Metric
- C11: renamed from C12; footprint (none) -> Capacitor_SMD:C_0603_1608Metric; now fitted
- C12: renamed from C10; footprint (none) -> Capacitor_SMD:C_0805_2012Metric
- C13: renamed from C11; footprint (none) -> Capacitor_SMD:C_0603_1608Metric
- C14: renamed from C3; footprint (none) -> Capacitor_SMD:C_0603_1608Metric
- C15: renamed from C4; footprint (none) -> Capacitor_SMD:C_0603_1608Metric
- C18: renamed from C16; value 10n -> 0.1u; footprint (none) -> Capacitor_SMD:C_0603_1608Metric
- C2: renamed from C15; value 50u -> 22u; footprint (none) -> Capacitor_SMD:CP_Elec_6.3x7.7
- C3: renamed from C13; footprint (none) -> Capacitor_SMD:C_0805_2012Metric
- C4: renamed from C14; value 0.1u -> 1u; footprint (none) -> Capacitor_SMD:C_0603_1608Metric
- C5: renamed from C2; footprint (none) -> Capacitor_SMD:C_0603_1608Metric
- C6: renamed from C5; value 0.1u -> 1u; footprint (none) -> Capacitor_SMD:C_0603_1608Metric
- C7: renamed from C6; value 1u -> 4.7u; footprint (none) -> Capacitor_SMD:C_0805_2012Metric
- C8: value 10u -> 4.7u; footprint (none) -> Capacitor_SMD:C_0805_2012Metric
- J1: renamed from J4; value +12V -> MAIN_IN
- J2: renamed from J3; value UPS Battery Connector -> AUX_IN
- J3: renamed from J5; value +12V_OUT -> VOUT
- L1: footprint (none) -> Inductor_SMD:L_APV_APH0850
- R1: renamed from R8; footprint (none) -> Resistor_SMD:R_0603_1608Metric
- R10: renamed from R25; footprint (none) -> Resistor_SMD:R_0603_1608Metric
- R11: renamed from R26; footprint (none) -> Resistor_SMD:R_0603_1608Metric
- R12: renamed from R15; footprint (none) -> Resistor_SMD:R_0603_1608Metric
- R13: renamed from R21; footprint (none) -> Resistor_SMD:R_0603_1608Metric
- R14: renamed from R22; footprint (none) -> Resistor_SMD:R_0603_1608Metric
- R15: renamed from R23; footprint (none) -> Resistor_SMD:R_0603_1608Metric
- R16: renamed from R24; footprint (none) -> Resistor_SMD:R_0603_1608Metric
- R17: renamed from R18; value 18.2k -> 3k; footprint (none) -> Resistor_SMD:R_0603_1608Metric
- R19: renamed from R12; footprint (none) -> Resistor_SMD:R_0603_1608Metric
- R2: renamed from R9; footprint (none) -> Resistor_SMD:R_0603_1608Metric
- R20: renamed from R17; value 15k -> 4.3k; footprint (none) -> Resistor_SMD:R_0603_1608Metric
- R3: renamed from R1; footprint (none) -> Resistor_SMD:R_1206_3216Metric
- R4: renamed from R2; footprint (none) -> Resistor_SMD:R_0603_1608Metric
- R5: renamed from R3; footprint (none) -> Resistor_SMD:R_0603_1608Metric
- R6: renamed from R5; footprint (none) -> Resistor_SMD:R_0603_1608Metric
- R7: renamed from R4; footprint (none) -> Resistor_SMD:R_0603_1608Metric
- R8: renamed from R13; value 18.2k -> 18k; footprint (none) -> Resistor_SMD:R_0603_1608Metric
- R9: renamed from R16; value 10k -> 15k; footprint (none) -> Resistor_SMD:R_0603_1608Metric
- renumbered D13 to D1, D10 to D3, D11 to D4, D12 to D5, Q7 to Q1, Q4 to Q2, Q5 to Q3, Q6 to Q4, Q3 to Q5, TP2 to TP1, TP3 to TP2
Connections:
- net AUX is gone; now on net +12V_AUX: C11.1, J2.2 (Pin_2), R3.2, R4.2, U1.13 (ISN)
- net +12V_AUX: now also C19.2, D6.1 (K), R18.2, TP11.1; no longer C11.2, C6.2, C7.2, C8.2, R3.1, U1.11 (VOUT), U1.12 (ISP)
- net +12V_OUT: now also C17.1, TP7.1
- net +5V_INT: now also TP4.1
- net GND: now also C10.2, C16.1, C17.2, C19.1, C9.1, D2.2 (A), D6.2 (A), H1.1, H2.1, H3.1, H4.1, R21.1; no longer J2.1 (Pin_1), R1.2
- net PG: now also TP9.1
- net STATUS: now also TP8.1
- net ~{CC}: now also TP10.1
- net SW1: now reaches C1.2, L1.1, TP1.1, U1.8 (SW1)
- net SW2: now reaches C5.2, L1.2, TP2.1, U1.10 (SW2)
- net EN/UVLO: now reaches R1.1, R2.2, U1.1 (EN_UVLO)
- net EN/UVLO: now also TP3.1
- net CP2: now reaches U2.3 (CP2)
- net CP2: now also R18.1, R21.2
- net FB: now reaches R4.1, R5.2, U1.14 (FB)
- net FB: now also TP5.1
- net COMP: now reaches C14.2, R7.2, U1.15 (COMP)
- net DITH_SYNC: now reaches C13.2, U1.5 (DITH_SYNC)
- net FSW: now reaches R6.2, U1.6 (FSW)
- net PR1: now reaches R17.2, R8.1, U2.6 (PR1)
- net +12V renamed +12V_MAIN
- net +12V_MAIN: now also R1.2, C16.2, D2.1 (K), TP6.1
- new net AUX-: J2.1 (Pin_1)
- new net ISP: C10.1, C11.2, C6.2, C7.2, C8.2, C9.2, R3.1, U1.11 (VOUT), U1.12 (ISP)
Other:
- added sheet Microcontroller (microcontroller.kicad_sch)
- note added: ">90% Output (Power Good)"
- note added: "Auxiliary Power"
- note added: "Backup VRLA"
- note added: "CHECK GATE THRESHOLD"
- note added: "Charger LEDs"
- note added: "Charging Circuit"
- note added: "Connectors"
- note added: "I_{LM} = 2.0 A"
- note added: "I_{LM} = 4.5 A"
- note added: "LVS Power"
- note added: "MAIN (IN1) is prioritised. Switches to AUX (IN2) if V_{MAIN} drops below ~11.4V. (Switchover: V_{PR1} < V_{CP2} -> 1.57V < 1.63V)"
- note added: "Main Power"
- note added: "Power MUX"
- note added: "ST = HIGH -> IN1 (MAIN) selected -> "MAIN" LED ON ST = LOW -> IN2 (AUX) selected -> "AUX" LED ON"
- note added: "Supply Status:"
- note added: "Switchover Logic:"
- note added: "TSAL UPS"
- note added: "To TSAL Logic"
- note added: "VOUT (+12V)"
- note added: "V_{IN1} = 10 V, V_{PR1} = 1.43"
- note added: "V_{IN1} = 11 V, V_{PR1} = 1.57"
- note added: "V_{IN1} = 12.7 V, V_{PR1} = 1.81"
- note added: "V_{IN2} = 11 V, V_{CP2} = 1.32 V"
- note added: "V_{IN2} = 12.7 V, V_{CP2} = 1.54 V"
- note added: "V_{IN2} = 13.5 V, V_{CP2} = 1.63 V"
- note added: "V_{OUT} = 13.5 V"
- note added: "V_{PR1} < V_{CP2} for IN2"
- note added: "V_{PR1} > V_{CP2} for IN1"
- note added: "WEBENCH® POWER DESIGNER"
- note added: "Yuasa NP0.8-12"
- note added: "falstad simulator"
- note added: "~400 kHz"
- note removed: ">90% Charged"
- company: (none) -> York Formula Student
- title: (none) -> TSAL UPS
- moved on the sheet: C1, C12, C13, C14, C15, C18, C2, C3, C4, C5, C6, C7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
